File: hardware/phaseA/phaseA.kicad_pcb (KiCad board)
At the start: 2 copper layers, 160 x 50 mm, 39 parts, among them K1 AQY212GH, U1 TXS0108EPWR, U2 TXS0108EPWR, U3 TXS0108EPWR, U4 TXS0108EPWR, U5 TXS0108EPWR, U6 TXS0108EPWR, U7 LM393

Commit message: Spec carte: platine clavier Atmos d'origine réutilisée telle quelle (matrice passive, scan par Pico #2)
Parts:
- moved R7 11.7 mm to (21.0, 27.0)
- moved J_PWR 10.9 mm to (10.0, 2.10)
- moved R1 8.60 mm to (33.0, 20.0)
- moved R2 8.60 mm to (36.0, 20.0)
- moved C15 5.00 mm to (21.0, 13.0)
- moved K1 3.00 mm to (21.0, 21.0)

Commit message: Phase B: gabarit acté = OriClone-1 (206,5x138 mm, trous extraits du .brd Eagle)
- Boîtier: OriClone-1 Case imprimable (Thingiverse 6228328, CC-BY-SA),
  STL mesurés 284x205 mm
- Référence matérielle clonée: hardware/oriclone-1-ref (JennyDigital,
  carte mère Eagle + platine clavier MX 'Oric Tactile KB' avec gerbers)
- Clavier de reconstruction disponible tel quel dans la référence
Parts:
- moved J_PRN 2.54 mm to (84.0, 7.04), turned to 90 degrees
- moved J_ULX_A 2.54 mm to (14.0, 46.5), turned to 90 degrees
- moved J_ULX_B 2.54 mm to (72.0, 46.5), turned to 90 degrees
